Commit message: Removed the collisions.

File: worm_picker_description/urdf/gp4_macro.xacro (robot description, xacro)
@@ -11,9 +11,9 @@
         <xacro:material_yaskawa_blue/>
       </visual>
-      <collision>
+      <!-- <collision>
         <geometry>
           <mesh filename="package://worm_picker_description/meshes/robot/collision/base_link.stl"/>
         </geometry>
-      </collision>
+      </collision> -->
     </link>
     <link name="${prefix}joint_1">
@@ -24,9 +24,9 @@
         <xacro:material_yaskawa_blue/>
       </visual>
-      <collision>
+      <!-- <collision>
         <geometry>
           <mesh filename="package://worm_picker_description/meshes/robot/collision/joint_1.stl"/>
         </geometry>
-      </collision>
+      </collision> -->
     </link>
     <link name="${prefix}joint_2">
@@ -37,9 +37,9 @@
         <xacro:material_yaskawa_blue/>
       </visual>
-      <collision>
+      <!-- <collision>
         <geometry>
           <mesh filename="package://worm_picker_description/meshes/robot/collision/joint_2.stl"/>
         </geometry>
-      </collision>
+      </collision> -->
     </link>
     <link name="${prefix}joint_3">
@@ -50,9 +50,9 @@
         <xacro:material_yaskawa_blue/>
       </visual>
-      <collision>
+      <!-- <collision>
         <geometry>
           <mesh filename="package://worm_picker_description/meshes/robot/collision/joint_3.stl"/>
         </geometry>
-      </collision>
+      </collision> -->
     </link>
     <link name="${prefix}joint_4">
@@ -63,9 +63,9 @@
         <xacro:material_yaskawa_blue/>
       </visual>
-      <collision>
+      <!-- <collision>
         <geometry>
           <mesh filename="package://worm_picker_description/meshes/robot/collision/joint_4.stl"/>
         </geometry>
-      </collision>
+      </collision> -->
     </link>
     <link name="${prefix}joint_5">
@@ -76,9 +76,9 @@
         <xacro:material_yaskawa_blue/>
       </visual>
-      <collision>
+      <!-- <collision>
         <geometry>
           <mesh filename="package://worm_picker_description/meshes/robot/collision/joint_5.stl"/>
         </geometry>
-      </collision>
+      </collision> -->
     </link>
     <link name="${prefix}joint_6">
@@ -89,9 +89,9 @@
         <xacro:material_yaskawa_silver/>
       </visual>
-      <collision>
+      <!-- <collision>
         <geometry>
           <mesh filename="package://worm_picker_description/meshes/robot/collision/joint_6.stl"/>
         </geometry>
-      </collision>
+      </collision> -->
     </link>
     <!-- end of link list -->
@@ -165,10 +165,10 @@
         </material>
       </visual>
-      <collision>
+      <!-- <collision>
         <origin xyz="0 0 0" rpy="0 0 0" />
         <geometry>
           <mesh filename="package://worm_picker_description/meshes/workcell/eoat_v2.stl"/>
         </geometry>
-      </collision>
+      </collision> -->
     </link>
     <joint name="flange-${prefix}eoat" type="fixed">
@@ -180,5 +180,5 @@
     <link name="${prefix}eoat_tcp"/>
     <joint name="${prefix}eoat-${prefix}eoat_tcp" type="fixed">
-      <origin xyz="0.1 0 -0.1" rpy="${radians(180)} ${radians(0)} ${radians(90)}"/>
+      <origin xyz="0.079 0 -0.0925" rpy="${radians(0)} ${radians(-60.0)} ${radians(180)}"/>
       <parent link="${prefix}eoat"/>
       <child link="${prefix}eoat_tcp"/>

File: worm_picker_description/urdf/workcell_macro.xacro (robot description, xacro)
@@ -20,10 +20,10 @@
         </material>
       </visual>
-      <collision>
+      <!-- <collision>
         <origin xyz="0 0 0" rpy="0 0 0" />
         <geometry>
           <mesh filename="package://worm_picker_description/meshes/workcell/workstation_v1_visual.stl"/>
         </geometry>
-      </collision>
+      </collision> -->
     </link>
     <joint name="world-workstation" type="fixed">
@@ -33,5 +33,5 @@
     </joint>
     <!-- Hotel 1 -->
-    <!-- <link name="hotel_1">
+    <link name="hotel_1">
       <visual>
         <origin xyz="0 0 0" rpy="0 0 0" />
@@ -43,16 +43,16 @@
         </material>
       </visual>
-      <collision>
+      <!-- <collision>
         <origin xyz="0 0 0" rpy="0 0 0" />
         <geometry>
           <mesh filename="package://worm_picker_description/meshes/workcell/hotel_1.stl"/>
         </geometry>
-      </collision>
+      </collision> -->
     </link>
     <joint name="world-hotel_1" type="fixed">
-      <origin xyz="0 0 0" rpy="0 0 0"/> <!- STL has origin defined at robot base_link origin ->
+      <origin xyz="0 0 0" rpy="0 0 0"/>  <!-- STL has origin defined at robot base_link origin -->
       <parent link="world"/>
       <child link="hotel_1"/>
-    </joint> -->
+    </joint>
     <!-- Float Table URDF -->
     <link name="table">
@@ -64,10 +64,10 @@
         </geometry>
       </visual>
-      <collision>
+      <!-- <collision>
         <origin xyz="0.9144 0 -0.1" rpy="0 0 0"/>
         <geometry>
           <box size="1.8288 1.2192 0.2"/>
         </geometry>
-      </collision>
+      </collision> -->
     </link>
     <joint name="world-table" type="fixed">
@@ -78,10 +78,10 @@
     <!-- Rough Collision Block - Ceiling -->
     <link name="ceiling">
-      <collision>
+      <!-- <collision>
         <origin xyz="0 0 0" rpy="0 0 0" />
         <geometry>
           <cylinder length="0.01" radius="3" />
         </geometry>
-      </collision>
+      </collision> -->
     </link>
     <joint name="world-ceiling" type="fixed">

Commit message: Update robot configuration: Modify defined stages parameters, adjust launch file paths, and enhance URDF structure for wormpick integration

File: worm_picker_description/urdf/gp4_macro.xacro (robot description, xacro)
@@ -140,5 +140,5 @@
     </joint>
     <!-- end of joint list -->
-    <!-- ROS-Industrial 'flange' frame -->
+    <!-- 'flange' frame -->
     <link name="${prefix}flange"/>
     <joint name="${prefix}joint_6-flange" type="fixed">
@@ -146,11 +146,4 @@
       <parent link="${prefix}joint_6"/>
       <child link="${prefix}flange"/>
-    </joint>
-    <!-- ROS-Industrial 'tool0' frame -->
-    <link name="${prefix}tool0"/>
-    <joint name="${prefix}flange-tool0" type="fixed">
-      <origin xyz="0 0 0" rpy="${radians(180)} ${radians(-90)} 0"/>
-      <parent link="${prefix}flange"/>
-      <child link="${prefix}tool0"/>
     </joint>
     <!-- End Effector -->
@@ -184,4 +177,18 @@
       <child link="${prefix}eoat_tcp"/>
     </joint>
+    <!-- WORMPICK -->
+    <link name="${prefix}wormpick"/>
+    <joint name="${prefix}flange-wormpick" type="fixed">
+      <origin xyz="0 0 0" rpy="${radians(0)} ${radians(0)} ${radians(0)}"/>
+      <parent link="${prefix}flange"/>
+      <child link="${prefix}wormpick"/>
+    </joint>
+    <!-- WORMPICK TCP -->
+    <link name="${prefix}wormpick_tcp"/>
+    <joint name="${prefix}wormpick-${prefix}wormpick_tcp" type="fixed">
+      <origin xyz="-0.05 -0.15 0.00" rpy="${radians(-90.0)} ${radians(0.0)} ${radians(0.0)}"/>
+      <parent link="${prefix}wormpick"/>
+      <child link="${prefix}wormpick_tcp"/>
+    </joint>
     <!-- ROS base_link to Robot Manufacturer World Coordinates transform -->
     <link name="${prefix}base" />

Commit message: Add GenerateHoverWormPickTask and update robot configuration: Introduce new task generator, modify workspace data, and enhance end effector definitions

File: worm_picker_description/urdf/gp4_macro.xacro (robot description, xacro)
@@ -165,29 +165,56 @@
       </collision> -->
     </link>
-    <joint name="flange-${prefix}eoat" type="fixed">
-      <origin xyz="0 0 0" rpy="0 0 0"/>
-      <parent link="flange"/>
-      <child link="${prefix}eoat"/>
+    <joint name="${prefix}flange-eoat" type="fixed">
+        <origin xyz="0 0 0" rpy="0 0 0"/>
+        <parent link="${prefix}flange"/>
+        <child link="${prefix}eoat"/>
     </joint>
     <!-- EOAT TCP -->
-    <link name="${prefix}eoat_tcp"/>
-    <joint name="${prefix}eoat-${prefix}eoat_tcp" type="fixed">
-      <origin xyz="0.079 0 -0.0925" rpy="${radians(0)} ${radians(-60.0)} ${radians(180)}"/>
-      <parent link="${prefix}eoat"/>
-      <child link="${prefix}eoat_tcp"/>
+    <link name="${prefix}eoat_tcp">
+        <visual>
+            <geometry>
+                <sphere radius="0.001"/>
+            </geometry>
+            <material name="red">
+                <color rgba="1 0 0 0.5"/>
+            </material>
+        </visual>
+    </link>
+    <joint name="${prefix}eoat-eoat_tcp" type="fixed">
+        <origin xyz="0.079 0 -0.0925" rpy="${radians(0)} ${radians(-60.0)} ${radians(180)}"/>
+        <parent link="${prefix}eoat"/>
+        <child link="${prefix}eoat_tcp"/>
     </joint>
     <!-- WORMPICK -->
-    <link name="${prefix}wormpick"/>
+    <link name="${prefix}wormpick">
+        <visual>
+            <geometry>
+                <box size="0.01 0.01 0.01"/>
+            </geometry>
+            <material name="blue">
+                <color rgba="0 0 1 0.5"/>
+            </material>
+        </visual>
+    </link>
     <joint name="${prefix}flange-wormpick" type="fixed">
-      <origin xyz="0 0 0" rpy="${radians(0)} ${radians(0)} ${radians(0)}"/>
-      <parent link="${prefix}flange"/>
-      <child link="${prefix}wormpick"/>
+        <origin xyz="0 0 0" rpy="${radians(0)} ${radians(0)} ${radians(0)}"/>
+        <parent link="${prefix}flange"/>
+        <child link="${prefix}wormpick"/>
     </joint>
     <!-- WORMPICK TCP -->
-    <link name="${prefix}wormpick_tcp"/>
-    <joint name="${prefix}wormpick-${prefix}wormpick_tcp" type="fixed">
-      <origin xyz="-0.05 -0.15 0.00" rpy="${radians(-90.0)} ${radians(0.0)} ${radians(0.0)}"/>
-      <parent link="${prefix}wormpick"/>
-      <child link="${prefix}wormpick_tcp"/>
+    <link name="${prefix}wormpick_tcp">
+        <visual>
+            <geometry>
+                <sphere radius="0.001"/>
+            </geometry>
+            <material name="green">
+                <color rgba="0 1 0 0.5"/>
+            </material>
+        </visual>
+    </link>
+    <joint name="${prefix}wormpick-wormpick_tcp" type="fixed">
+        <origin xyz="-0.05 -0.15 0.00" rpy="${radians(-90.0)} ${radians(0.0)} ${radians(0.0)}"/>
+        <parent link="${prefix}wormpick"/>
+        <child link="${prefix}wormpick_tcp"/>
     </joint>
     <!-- ROS base_link to Robot Manufacturer World Coordinates transform -->

File: worm_picker_moveit_config/config/worm_picker_robot.urdf.xacro (robot description, xacro)
@@ -1,11 +1,11 @@
 <?xml version="1.0"?>
 <robot xmlns:xacro="http://ros.org/wiki/xacro" name="worm_picker_robot">
-  <xacro:arg name="initial_positions_file" default="$(find worm_picker_moveit_config)/config/initial_positions.yaml" />
+  <!-- <xacro:arg name="initial_positions_file" default="$(find worm_picker_moveit_config)/config/initial_positions.yaml" /> -->
   <!-- Include necessary Xacro files -->
   <xacro:include filename="$(find worm_picker_description)/urdf/worm_picker_robot.urdf.xacro" />
-  <xacro:include filename="$(find worm_picker_moveit_config)/config/worm_picker_robot.ros2_control.xacro" />
+  <!-- <xacro:include filename="$(find worm_picker_moveit_config)/config/worm_picker_robot.ros2_control.xacro" /> -->
   <!-- Instantiate the ROS 2 control macro -->
-  <xacro:worm_picker_robot_ros2_control
+  <!-- <xacro:worm_picker_robot_ros2_control
     name="FakeSystem"
-    initial_positions_file="$(arg initial_positions_file)" />
+    initial_positions_file="$(arg initial_positions_file)" /> -->
 </robot>

Commit message: Add FixedPoint and WorkstationGeometry data types, and update PlatePositionAnalyzer: Introduce FixedPoint and WorkstationGeometry structs, refactor PlatePositionAnalyzer to utilize these new data types, and enhance quaternion handling for pose transformations.

File: worm_picker_description/urdf/gp4_macro.xacro (robot description, xacro)
@@ -183,4 +183,5 @@
     <joint name="${prefix}eoat-eoat_tcp" type="fixed">
         <origin xyz="0.079 0 -0.0925" rpy="${radians(0)} ${radians(-60.0)} ${radians(180)}"/>
+        <!-- <origin xyz="0.079 0 -0.0925" rpy="${radians(0)} ${radians(-60.0)} ${radians(0)}"/> This is more correct, need to change later -->
         <parent link="${prefix}eoat"/>
         <child link="${prefix}eoat_tcp"/>

Commit message: Update copyright year to 2025 and adjust motion parameters for improved task execution

File: worm_picker_description/urdf/gp4_macro.xacro (robot description, xacro)
@@ -182,5 +182,5 @@
     </link>
     <joint name="${prefix}eoat-eoat_tcp" type="fixed">
-        <origin xyz="0.079 0 -0.0925" rpy="${radians(0)} ${radians(-60.0)} ${radians(180)}"/>
+        <origin xyz="0.11024 0.00 -0.07075" rpy="${radians(180)} ${radians(-150.0)} ${radians(180)}"/>
         <parent link="${prefix}eoat"/>
         <child link="${prefix}eoat_tcp"/>

Commit message: Modifying urdf files for new wormpick

File: worm_picker_description/urdf/gp4_macro.xacro (robot description, xacro)
@@ -214,5 +214,5 @@
     </link>
     <joint name="${prefix}wormpick-wormpick_tcp" type="fixed">
-        <origin xyz="-0.05 -0.15 0.00" rpy="${radians(-90.0)} ${radians(0.0)} ${radians(0.0)}"/>
+        <origin xyz="-0.065 -0.15 0.00" rpy="${radians(-90.0)} ${radians(0.0)} ${radians(0.0)}"/>
         <parent link="${prefix}wormpick"/>
         <child link="${prefix}wormpick_tcp"/>

Commit message: moddifying worm pick hover offset and urdf

File: worm_picker_description/urdf/gp4_macro.xacro (robot description, xacro)
@@ -214,5 +214,5 @@
     </link>
     <joint name="${prefix}wormpick-wormpick_tcp" type="fixed">
-        <origin xyz="-0.065 -0.15 0.00" rpy="${radians(-90.0)} ${radians(0.0)} ${radians(0.0)}"/>
+        <origin xyz="-0.075 -0.15 0.005" rpy="${radians(-90.0)} ${radians(0.0)} ${radians(0.0)}"/>
         <parent link="${prefix}wormpick"/>
         <child link="${prefix}wormpick_tcp"/>

Commit message: z value for wormpick-wormpick_tcp must be 0 otherwise planing traj fail probably due to the fast spin issue

File: worm_picker_description/urdf/gp4_macro.xacro (robot description, xacro)
@@ -214,5 +214,5 @@
     </link>
     <joint name="${prefix}wormpick-wormpick_tcp" type="fixed">
-        <origin xyz="-0.075 -0.15 0.005" rpy="${radians(-90.0)} ${radians(0.0)} ${radians(0.0)}"/>
+        <origin xyz="-0.075 -0.15 0.000" rpy="${radians(-90.0)} ${radians(0.0)} ${radians(0.0)}"/>
         <parent link="${prefix}wormpick"/>
         <child link="${prefix}wormpick_tcp"/>
